File: KiCadProjects/Example_Design/Example_Design.kicad_pcb (KiCad board)
At the start: 2 copper layers, 38.1 x 31.8 mm, 15 parts, among them J1 DT13-6P

Commit message: Add files via upload
Other:
- net class Default removed
