File: KiCadProjects/add-sub-module/add-sub-module.kicad_sch (KiCad schematic)
At the start: 0 parts

Commit message: Working on add-sub schematic
Parts:
- added U1: CD74HCT10E, footprints.pretty3:N14, symbol 2024-10-26_20-42-17:CD74HCT10E
- added U2: SN74HCT00N, footprints.pretty6:N14, symbol 2024-10-26_20-41-17:SN74HCT00N
- added U3: SN74HCT02N, footprints.pretty7:N14, symbol 2024-10-23_21-39-10:SN74HCT02N
- added U4: SN74HCT257N, footprints.pretty8:N16, symbol 2024-10-23_21-18-01:SN74HCT257N
- added U5: CD74HCT04E, footprints.pretty1:N14, symbol 2024-10-26_20-41-30:CD74HCT04E
Connections:
- new net: U1.10 (3B), U2.5 (2B), U2.9 (3A), U3.12 (4B), U3.2 (1A), U5.10 (*5Y)
- new net: U3.10 (3Y), U5.11 (5A)
- new net: U3.4 (2Y), U5.13 (6A)
- new net: U1.2 (1B), U3.8 (3A), U5.2 (*1Y)
- new net: U1.1 (1A), U3.9 (3B), U5.4 (*2Y)
- new net: U1.3 (2A), U5.6 (*3Y), U5.9 (4A)
- new net: U1.9 (3A), U2.12 (4A), U5.8 (*4Y)
- new net: U3.1 (1Y), U4.2 (1A)
- new net: U3.13 (4Y), U4.13 (4B)
- new net: U3.5 (2A), U4.12 (4Y)
- new net: U3.6 (2B), U4.4 (1Y)
- new net +5V: U1.14 (VCC), U2.14 (VCC), U3.14 (VCC), U4.16 (VCC), U5.14 (VCC)
- new net Cin: U5.1 (1A)
- new net Cout: U5.12 (*6Y)
- new net X: U5.5 (3A)
- new net Y: U5.3 (2A)
Other:
- note added: "Hex NOT"
- note added: "Quad 2-1 MUX"
- note added: "Quad 2-Input NAND"
- note added: "Quad 2-Input NOR"
- note added: "Tri 3-Input NAND"

Commit message: Finished add-sub schematic
Connections:
- net +5V: now also U1.13 (1C)
- net at U1.10 (3B), U2.5 (2B), U2.9 (3A)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: now also U1.4 (2B)
- net at U1.11 (3C): now also U1.12 (1Y), U1.5 (2C)
- net at U1.6 (2Y): now also U2.2 (1B), U2.4 (2A), U3.3 (1B)
- net at U1.8 (3Y): now also U2.10 (3B), U2.13 (4B), U3.11 (4A)
- net at U2.1 (1A): now also U2.11 (4Y)
- net S: now reaches U2.3 (1Y)
- net at U2.6 (2Y): now also U4.3 (1B)
- net at U2.8 (3Y): now also U4.14 (4A)
- net ~A/S: now reaches U4.1 (*A/B)
Other:
- moved on the sheet: U1, U2, U3, U4, U5

Commit message: rev. v1 for add sub
Parts:
- added C1, C2, C3, C4, C5: 0.1 uF, Capacitor_THT:C_Disc_D4.7mm_W2.5mm_P5.00mm, symbol Device:C
- added D1, D2, D3, D4, D5, D6: D, LED_THT:LED_D5.0mm, symbol Device:D
- added J1: 2x4_Header, 0_add_sub:2x4_Header, symbol 0_add_sub:2x4_Header
- added J2: 1x2_Header, 0_add_sub:1x2_Header, symbol 0_add_sub:1x2_Header
- added R1, R2, R3, R4, R5, R6: 1k, Resistor_THT:R_Axial_DIN0207_L6.3mm_D2.5mm_P7.62mm_Horizontal, symbol Device:R
- U1: footprint footprints.pretty3:N14 -> 0_add_sub:DIP_14; symbol 2024-10-26_20-42-17:CD74HCT10E -> 0_add_sub:CD74HCT10E; LCSC (none) -> CD74HCT10E; Link (none) -> https://www.digikey.com/en/products/detail/texas-instrument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; Part No (none) -> 296-2086-5-ND
- U2: footprint footprints.pretty6:N14 -> 0_add_sub:DIP_14; symbol 2024-10-26_20-41-17:SN74HCT00N -> 0_add_sub:SN74HCT00N; LCSC (none) -> SN74HCT00N; Link (none) -> https://www.digikey.com/en/products/detail/texas-instrument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; Part No (none) -> 296-1603-5-ND
- U3: footprint footprints.pretty7:N14 -> 0_add_sub:DIP_14; symbol 2024-10-23_21-39-10:SN74HCT02N -> 0_add_sub:SN74HCT02N; LCSC (none) -> SN74HCT02N; Link (none) -> https://www.digikey.com/en/products/detail/texas-instrument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; Part No (none) -> 296-8380-5-ND
- U4: footprint footprints.pretty8:N16 -> 0_add_sub:DIP_16; symbol 2024-10-23_21-18-01:SN74HCT257N -> 0_add_sub:SN74HCT257N; LCSC (none) -> SN74HCT257N; Link (none) -> https://www.digikey.com/en/products/detail/texas-instrument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; Part No (none) -> 296-8406-5-ND
- U5: footprint footprints.pretty1:N14 -> 0_add_sub:DIP_14; symbol 2024-10-26_20-41-30:CD74HCT04E -> 0_add_sub:CD74HCT04E; LCSC (none) -> CD74HCT04E; Link (none) -> https://www.digikey.com/en/products/detail/texas-instrument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; Part No (none) -> 296-2083-5-ND
Connections:
- net +5V: now also U4.15 (*OE), C1.1, C2.1, C3.1, C4.1, C5.1, J1.1
- net GND: now reaches U5.7 (GND)
- net GND: now also U1.7 (GND), U2.7 (GND), U3.7 (GND), U4.10 (3B), U4.11 (3A), U4.5 (2A), U4.6 (2B), U4.8 (GND), C1.2, C2.2, C3.2, C4.2, C5.2, J1.7, R1.2, R2.2, R3.2, R4.2, R5.2, R6.2
- net Cin renamed CARRY
- net CARRY: now also D1.2 (A), J1.8
- net Cout renamed COUT
- net COUT: now also D6.2 (A), J2.2
- net S renamed SUM
- net SUM: now also D5.2 (A), J2.1
- net X renamed CA
- net CA: now also D3.2 (A), J1.4
- net Y renamed KA
- net KA: now also D2.2 (A), J1.2
- net ~A/S renamed ADD/SUB
- net ADD/SUB: now also D4.2 (A), J1.6
- new net: D4.1 (K), R4.1
- new net: D3.1 (K), R3.1
- new net: D2.1 (K), R2.1
- new net: D5.1 (K), R5.1
- new net: D1.1 (K), R1.1
- new net: D6.1 (K), R6.1
- new net CLK: J1.5
- new net RST: J1.3
- no-connect marks 0 -> 2

Commit message: finished tester design
Connections:
- net +5V: now also J1.2; no longer J1.1
- net ADD/SUB: now also J1.5; no longer J1.6
- net CA: now also J1.3; no longer J1.4
- net CARRY: now also J1.7; no longer J1.8
- net CLK: now also J1.6; no longer J1.5
- net GND: now also J1.8; no longer J1.7
- net KA: now also J1.1; no longer J1.2
- net RST: now also J1.4; no longer J1.3

Commit message: Updated links and footprints in add-subtractor schematic, also added my maker's mark
Parts:
- C1, C2, C3, C4, C5: Link (none) -> https://jlcpcb.com/partdetail/85943-CT40805B104K500F3/C84772; Part No (none) -> C84772
- J1: footprint 0_add_sub:2x4_Header -> Connector_PinHeader_2.54mm:PinHeader_2x04_P2.54mm_Vertical; Link https://www.digikey.com/en/products/detail/samtec-inc/TSW-1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 -> https://jlcpcb.com/partdetail/Samtec-TSW_104_07_FD/C6339738; Part No SAM8996-ND -> C6339738
- J2: footprint 0_add_sub:1x2_Header -> Connector_PinHeader_2.54mm:PinHeader_1x02_P2.54mm_Vertical; Link https://www.digikey.com/en/products/detail/samtec-inc/TSW-1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 -> https://jlcpcb.com/partdetail/Samtec-TSW_102_23_FS/C3329876; Part No SAM10326-ND -> C3329876
- U1: footprint 0_add_sub:DIP_14 -> Package_DIP:DIP-14_W7.62mm; Link https://www.digikey.com/en/products/detail/texas-instrument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 -> https://jlcpcb.com/partdetail/TexasInstruments-CD74HCT10E/C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; Part No 296-2086-5-ND -> C2862275
- U2: footprint 0_add_sub:DIP_14 -> Package_DIP:DIP-14_W7.62mm; Link https://www.digikey.com/en/products/detail/texas-instrument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 -> https://jlcpcb.com/partdetail/TexasInstruments-SN74HCT00N/C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; Part No 296-1603-5-ND -> C354416
- U3: footprint 0_add_sub:DIP_14 -> Package_DIP:DIP-14_W7.62mm; Link https://www.digikey.com/en/products/detail/texas-instrument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 -> https://jlcpcb.com/partdetail/TexasInstruments-SN74HCT02N/C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; Part No 296-8380-5-ND -> C354417
- U4: footprint 0_add_sub:DIP_16 -> Package_DIP:DIP-16_W7.62mm; Link https://www.digikey.com/en/products/detail/texas-instrument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 -> https://jlcpcb.com/partdetail/TexasInstruments-SN74HCT257N/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; Part No 296-8406-5-ND -> C1547251
- U5: footprint 0_add_sub:DIP_14 -> Package_DIP:DIP-14_W7.62mm; Link https://www.digikey.com/en/products/detail/texas-instrument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 -> https://jlcpcb.com/partdetail/TexasInstruments-CD74HCT04E/C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; Part No 296-2083-5-ND -> C2879109
Changed lines of the file:
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@@
 			)
 		)
-		(property "Part No" ""
+		(property "Part No" "C84772"
 			(at 22.86 49.53 0)
 			(effects
@@
 			)
 		)
-		(property "Link" ""
+		(property "Link" "https://jlcpcb.com/partdetail/85943-CT40805B104K500F3/C84772"
 			(at 22.86 49.53 0)
 			(effects
@@
 			)
 		)
-		(property "Footprint" "0_add_sub:DIP_14"
+		(property "Footprint" "Package_DIP:DIP-14_W7.62mm"
 			(at 231.14 114.3 0)
 			(effects
@@
 			)
 		)
-		(property "Part No" "296-2083-5-ND"
+		(property "Part No" "C2879109"
 			(at 231.14 114.3 0)
 			(effects
@@
 			)
 		)
-		(property "Link" "https://www.digikey.com/en/products/detail/texas-instruments/CD74HCT04E/38238"
+		(property "Link" "https://jlcpcb.com/partdetail/TexasInstruments-CD74HCT04E/C2879109"
 			(at 231.14 114.3 0)
 			(effects
@@
 			)
 		)
-		(property "Part No" ""
+		(property "Part No" "C84772"
 			(at 22.86 92.71 0)
 			(effects
@@
 			)
 		)
-		(property "Link" ""
+		(property "Link" "https://jlcpcb.com/partdetail/85943-CT40805B104K500F3/C84772"
 			(at 22.86 92.71 0)
 			(effects
@@
 			)
 		)
-		(property "Footprint" "0_add_sub:1x2_Header"
+		(property "Footprint" "Connector_PinHeader_2.54mm:PinHeader_1x02_P2.54mm_Vertical"
 			(at 30.48 186.69 0)
 			(effects
@@
 			)
 		)
-		(property "Part No" "SAM10326-ND"
+		(property "Part No" "C3329876"
 			(at 30.48 186.69 0)
 			(effects
@@
 			)
 		)
-		(property "Link" "https://www.digikey.com/en/products/detail/samtec-inc/TSW-102-23-F-S/6679063"
+		(property "Link" "https://jlcpcb.com/partdetail/Samtec-TSW_102_23_FS/C3329876"
 			(at 30.48 186.69 0)
 			(effects
@@
 			)
 		)
-		(property "Footprint" "0_add_sub:DIP_14"
+		(property "Footprint" "Package_DIP:DIP-14_W7.62mm"
 			(at 40.64 114.3 0)
 			(effects
@@
 			)
 		)
-		(property "Part No" "296-2086-5-ND"
+		(property "Part No" "C2862275"
 			(at 40.64 114.3 0)
 			(effects
@@
 			)
 		)
-		(property "Link" "https://www.digikey.com/en/products/detail/texas-instruments/CD74HCT10E/38242?s=N4IgTCBcDaIMIBEDsAWAEnAKgRgAwFEQBdAXyA"
+		(property "Link" "https://jlcpcb.com/partdetail/TexasInstruments-CD74HCT10E/C2862275"
 			(at 40.64 114.3 0)
 			(effects
@@
 			)
 		)
-		(property "Part No" ""
+		(property "Part No" "C84772"
 			(at 22.86 114.3 0)
 			(effects
@@
 			)
 		)
-		(property "Link" ""
+		(property "Link" "https://jlcpcb.com/partdetail/85943-CT40805B104K500F3/C84772"
 			(at 22.86 114.3 0)
 			(effects
@@
 			)
 		)
-		(property "Footprint" "0_add_sub:DIP_14"
+		(property "Footprint" "Package_DIP:DIP-14_W7.62mm"
 			(at 134.62 114.3 0)
 			(effects
@@
 			)
 		)
-		(property "Part No" "296-8380-5-ND"
+		(property "Part No" "C354417"
 			(at 134.62 114.3 0)
 			(effects
@@
 			)
 		)
-		(property "Link" "https://www.digikey.com/en/products/detail/texas-instruments/SN74HCT02N/376866"
+		(property "Link" "https://jlcpcb.com/partdetail/TexasInstruments-SN74HCT02N/C354417"
 			(at 134.62 114.3 0)
 			(effects
@@
 			)
 		)
-		(property "Footprint" "0_add_sub:DIP_14"
+		(property "Footprint" "Package_DIP:DIP-14_W7.62mm"
 			(at 86.36 114.3 0)
 			(effects
@@
 			)
 		)
-		(property "Part No" "296-1603-5-ND"
+		(property "Part No" "C354416"
 			(at 86.36 114.3 0)
 			(effects
@@
 			)
 		)
-		(property "Link" "https://www.digikey.com/en/products/detail/texas-instruments/SN74HCT00N/277249"
+		(property "Link" "https://jlcpcb.com/partdetail/TexasInstruments-SN74HCT00N/C354416"
 			(at 86.36 114.3 0)
 			(effects
@@
 			)
 		)
-		(property "Part No" ""
+		(property "Part No" "C84772"
 			(at 22.86 71.12 0)
 			(effects
@@
 			)
 		)
-		(property "Link" ""
+		(property "Link" "https://jlcpcb.com/partdetail/85943-CT40805B104K500F3/C84772"
 			(at 22.86 71.12 0)
 			(effects
@@
 			)
 		)
-		(property "Footprint" "0_add_sub:DIP_16"
+		(property "Footprint" "Package_DIP:DIP-16_W7.62mm"
 			(at 180.34 114.3 0)
 			(effects
@@
 			)
 		)
-		(property "Part No" "296-8406-5-ND"
+		(property "Part No" "C1547251"
 			(at 180.34 114.3 0)
 			(effects
@@
 			)
 		)
-		(property "Link" "https://www.digikey.com/en/products/detail/texas-instruments/SN74HCT257N/376803?s=N4IgTCBcDaIMoDkDsAWAEgYQCpgKxIRAF0BfIA"
+		(property "Link" "https://jlcpcb.com/partdetail/TexasInstruments-SN74HCT257N/C1547251"
 			(at 180.34 114.3 0)
 			(effects
@@
 			)
 		)
-		(property "Part No" ""
+		(property "Part No" "C84772"
 			(at 22.86 27.94 0)
 			(effects
@@
 			)
 		)
-		(property "Link" ""
+		(property "Link" "https://jlcpcb.com/partdetail/85943-CT40805B104K500F3/C84772"
 			(at 22.86 27.94 0)
 			(effects
@@
 			)
 		)
-		(property "Footprint" "0_add_sub:2x4_Header"
+		(property "Footprint" "Connector_PinHeader_2.54mm:PinHeader_2x04_P2.54mm_Vertical"
 			(at 30.48 160.02 0)
 			(effects
@@
 			)
 		)
-		(property "Part No" "SAM8996-ND"
+		(property "Part No" "C6339738"
 			(at 30.48 160.02 0)
 			(effects
@@
 			)
 		)
-		(property "Link" "https://www.digikey.com/en/products/detail/samtec-inc/TSW-104-07-F-D/2685891"
+		(property "Link" "https://jlcpcb.com/partdetail/Samtec-TSW_104_07_FD/C6339738"
 			(at 30.48 160.02 0)
 			(effects

Commit message: Changed footprints in schematic
Parts:
- C1, C2, C3, C4, C5: Link https://jlcpcb.com/partdetail/85943-CT40805B104K500F3/C84772 -> https://www.newark.com/multicomp/mc0805b104k500a5-08mm/cera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; Part No C84772 -> (none)
- U1: footprint Package_DIP:DIP-14_W7.62mm -> Package_DIP:DIP-14_W7.62mm_Socket; Link https://jlcpcb.com/partdetail/TexasInstruments-CD74HCT10E/C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 -> https://www.digikey.com/en/products/detail/texas-instrument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; Part No C2862275 -> (none)
- U2: footprint Package_DIP:DIP-14_W7.62mm -> Package_DIP:DIP-14_W7.62mm_Socket; Link https://jlcpcb.com/partdetail/TexasInstruments-SN74HCT00N/C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 -> https://www.digikey.com/en/products/detail/texas-instrument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; Part No C354416 -> (none)
- U3: footprint Package_DIP:DIP-14_W7.62mm -> Package_DIP:DIP-14_W7.62mm_Socket; Link https://jlcpcb.com/partdetail/TexasInstruments-SN74HCT02N/C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 -> https://www.digikey.com/en/products/detail/texas-instrument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; Part No C354417 -> (none)
- U4: footprint Package_DIP:DIP-16_W7.62mm -> Package_DIP:DIP-16_W7.62mm_Socket; Link https://jlcpcb.com/partdetail/TexasInstruments-SN74HCT257N/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 -> https://www.digikey.com/en/products/detail/texas-instrument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; Part No C1547251 -> (none)
- U5: footprint Package_DIP:DIP-14_W7.62mm -> Package_DIP:DIP-14_W7.62mm_Socket; Link https://jlcpcb.com/partdetail/TexasInstruments-CD74HCT04E/C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 -> https://www.digikey.com/en/products/detail/texas-instrument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; Part No C2879109 -> (none)
Changed lines of the file:
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@@
 			)
 		)
-		(property "Part No" "C84772"
+		(property "Part No" ""
 			(at 22.86 49.53 0)
 			(effects
@@
 			)
 		)
-		(property "Link" "https://jlcpcb.com/partdetail/85943-CT40805B104K500F3/C84772"
+		(property "Link" "https://www.newark.com/multicomp/mc0805b104k500a5-08mm/ceramic-capacitor-0-1uf-50v-x7r/dp/46P6240"
 			(at 22.86 49.53 0)
 			(effects
@@
 			)
 		)
-		(property "Footprint" "Package_DIP:DIP-14_W7.62mm"
+		(property "Footprint" "Package_DIP:DIP-14_W7.62mm_Socket"
 			(at 231.14 114.3 0)
 			(effects
@@
 			)
 		)
-		(property "Part No" "C2879109"
+		(property "Part No" ""
 			(at 231.14 114.3 0)
 			(effects
@@
 			)
 		)
-		(property "Link" "https://jlcpcb.com/partdetail/TexasInstruments-CD74HCT04E/C2879109"
+		(property "Link" "https://www.digikey.com/en/products/detail/texas-instruments/CD74HCT04E/38238"
 			(at 231.14 114.3 0)
 			(effects
@@
 			)
 		)
-		(property "Part No" "C84772"
+		(property "Part No" ""
 			(at 22.86 92.71 0)
 			(effects
@@
 			)
 		)
-		(property "Link" "https://jlcpcb.com/partdetail/85943-CT40805B104K500F3/C84772"
+		(property "Link" "https://www.newark.com/multicomp/mc0805b104k500a5-08mm/ceramic-capacitor-0-1uf-50v-x7r/dp/46P6240"
 			(at 22.86 92.71 0)
 			(effects
@@
 			)
 		)
-		(property "Footprint" "Package_DIP:DIP-14_W7.62mm"
+		(property "Footprint" "Package_DIP:DIP-14_W7.62mm_Socket"
 			(at 40.64 114.3 0)
 			(effects
@@
 			)
 		)
-		(property "Part No" "C2862275"
+		(property "Part No" ""
 			(at 40.64 114.3 0)
 			(effects
@@
 			)
 		)
-		(property "Link" "https://jlcpcb.com/partdetail/TexasInstruments-CD74HCT10E/C2862275"
+		(property "Link" "https://www.digikey.com/en/products/detail/texas-instruments/CD74HCT10E/38242"
 			(at 40.64 114.3 0)
 			(effects
@@
 			)
 		)
-		(property "Part No" "C84772"
+		(property "Part No" ""
 			(at 22.86 114.3 0)
 			(effects
@@
 			)
 		)
-		(property "Link" "https://jlcpcb.com/partdetail/85943-CT40805B104K500F3/C84772"
+		(property "Link" "https://www.newark.com/multicomp/mc0805b104k500a5-08mm/ceramic-capacitor-0-1uf-50v-x7r/dp/46P6240"
 			(at 22.86 114.3 0)
 			(effects
@@
 			)
 		)
-		(property "Footprint" "Package_DIP:DIP-14_W7.62mm"
+		(property "Footprint" "Package_DIP:DIP-14_W7.62mm_Socket"
 			(at 134.62 114.3 0)
 			(effects
@@
 			)
 		)
-		(property "Part No" "C354417"
+		(property "Part No" ""
 			(at 134.62 114.3 0)
 			(effects
@@
 			)
 		)
-		(property "Link" "https://jlcpcb.com/partdetail/TexasInstruments-SN74HCT02N/C354417"
+		(property "Link" "https://www.digikey.com/en/products/detail/texas-instruments/SN74HCT02N/376866"
 			(at 134.62 114.3 0)
 			(effects
@@
 			)
 		)
-		(property "Footprint" "Package_DIP:DIP-14_W7.62mm"
+		(property "Footprint" "Package_DIP:DIP-14_W7.62mm_Socket"
 			(at 86.36 114.3 0)
 			(effects
@@
 			)
 		)
-		(property "Part No" "C354416"
+		(property "Part No" ""
 			(at 86.36 114.3 0)
 			(effects
@@
 			)
 		)
-		(property "Link" "https://jlcpcb.com/partdetail/TexasInstruments-SN74HCT00N/C354416"
+		(property "Link" "https://www.digikey.com/en/products/detail/texas-instruments/SN74HCT00N/277249"
 			(at 86.36 114.3 0)
 			(effects
@@
 			)
 		)
-		(property "Part No" "C84772"
+		(property "Part No" ""
 			(at 22.86 71.12 0)
 			(effects
@@
 			)
 		)
-		(property "Link" "https://jlcpcb.com/partdetail/85943-CT40805B104K500F3/C84772"
+		(property "Link" "https://www.newark.com/multicomp/mc0805b104k500a5-08mm/ceramic-capacitor-0-1uf-50v-x7r/dp/46P6240"
 			(at 22.86 71.12 0)
 			(effects
@@
 			)
 		)
-		(property "Footprint" "Package_DIP:DIP-16_W7.62mm"
+		(property "Footprint" "Package_DIP:DIP-16_W7.62mm_Socket"
 			(at 180.34 114.3 0)
 			(effects
@@
 			)
 		)
-		(property "Part No" "C1547251"
+		(property "Part No" ""
 			(at 180.34 114.3 0)
 			(effects
@@
 			)
 		)
-		(property "Link" "https://jlcpcb.com/partdetail/TexasInstruments-SN74HCT257N/C1547251"
+		(property "Link" "https://www.digikey.com/en/products/detail/texas-instruments/SN74HCT257N/376803"
 			(at 180.34 114.3 0)
 			(effects
@@
 			)
 		)
-		(property "Part No" "C84772"
+		(property "Part No" ""
 			(at 22.86 27.94 0)
 			(effects
@@
 			)
 		)
-		(property "Link" "https://jlcpcb.com/partdetail/85943-CT40805B104K500F3/C84772"
+		(property "Link" "https://www.newark.com/multicomp/mc0805b104k500a5-08mm/ceramic-capacitor-0-1uf-50v-x7r/dp/46P6240"
 			(at 22.86 27.94 0)
 			(effects

Commit message: Fixed a couple links
Parts:
- J1: Link https://jlcpcb.com/partdetail/Samtec-TSW_104_07_FD/C6339738 -> https://www.digikey.com/en/products/detail/samtec-inc/TSW-1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
- J2: Link https://jlcpcb.com/partdetail/Samtec-TSW_102_23_FS/C3329876 -> https://www.digikey.com/en/products/detail/samtec-inc/TSW-1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
Changed lines of the file:
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@@
 			)
 		)
-		(property "Datasheet" ""
+		(property "Datasheet" "https://mm.digikey.com/Volume0/opasdata/d220001/medias/docus/6129/tsw-xxx-xx-xxx-x-xx-xxx-mkt.pdf"
 			(at 30.48 186.69 0)
 			(effects
@@
 			)
 		)
-		(property "Link" "https://jlcpcb.com/partdetail/Samtec-TSW_102_23_FS/C3329876"
+		(property "Link" "https://www.digikey.com/en/products/detail/samtec-inc/TSW-102-23-F-S/6679063"
 			(at 30.48 186.69 0)
 			(effects
@@
 			)
 		)
-		(property "Datasheet" ""
+		(property "Datasheet" "https://mm.digikey.com/Volume0/opasdata/d220001/medias/docus/6129/tsw-xxx-xx-xxx-x-xx-xxx-mkt.pdf"
 			(at 30.48 160.02 0)
 			(effects
@@
 			)
 		)
-		(property "Link" "https://jlcpcb.com/partdetail/Samtec-TSW_104_07_FD/C6339738"
+		(property "Link" "https://www.digikey.com/en/products/detail/samtec-inc/TSW-104-07-F-D/2685891"
 			(at 30.48 160.02 0)
 			(effects

Commit message: Adding socket part numbers to ICs in schematic
Parts:
- U1, U2, U3, U5: Part No (none) -> C2325
- U4: Part No (none) -> C2326
Changed lines of the file:
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@@
 			)
 		)
-		(property "Part No" ""
+		(property "Part No" "C2325"
 			(at 231.14 114.3 0)
 			(effects
@@
 			)
 		)
-		(property "Part No" ""
+		(property "Part No" "C2325"
 			(at 40.64 114.3 0)
 			(effects
@@
 			)
 		)
-		(property "Part No" ""
+		(property "Part No" "C2325"
 			(at 134.62 114.3 0)
 			(effects
@@
 			)
 		)
-		(property "Part No" ""
+		(property "Part No" "C2325"
 			(at 86.36 114.3 0)
 			(effects
@@
 			)
 		)
-		(property "Part No" ""
+		(property "Part No" "C2326"
 			(at 180.34 114.3 0)
 			(effects
