File: KiCadProjects/add-sub-module-tester/add-sub-module-tester.kicad_pcb (KiCad board)
At the start: 2 copper layers, 92 x 63 mm, 36 parts, among them J1 Conn_01x04_Socket, J2 Conn_01x04_Socket, J3 12V In, J4 Conn_01x02_Socket, SW1 PWR_SW, U1 Toggle_Switch_3PIN, U2 Toggle_Switch_3PIN, U3 Toggle_Switch_3PIN, U4 Toggle_Switch_3PIN, U5 AP6503

Commit message: FINAL final changes for Rev. A
Parts:
- D1: footprint LED_SMD:LED_0805_2012Metric_Pad1.15x1.40mm_HandSolder -> LED_SMD:LED_0603_1608Metric_Pad1.05x0.95mm_HandSolder
- moved REF** 39.0 mm to (156.5, 97.8)
Other:
- board text added: "+12VDC"
- board text removed: "CA"
- board text removed: "CARRY"
- board text removed: "KA"
Changed lines of the file:
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@@
 	(net 23 "unconnected-(J4-Pin_2-Pad2)")
 	(net 24 "unconnected-(J4-Pin_1-Pad1)")
-	(footprint "LED_SMD:LED_0805_2012Metric_Pad1.15x1.40mm_HandSolder"
+	(footprint "LED_SMD:LED_0603_1608Metric_Pad1.05x0.95mm_HandSolder"
 		(layer "F.Cu")
 		(at 129.5 91.5625 -90)
-		(descr "LED SMD 0805 (2012 Metric), square (rectangular) end terminal, IPC_7351 nominal, (Body size source: https://docs.google.com/spreadsheets/d/1BsfQQcO9C6DZCsRaXUlFlo91Tg2WpOkGARC1WS5S8t0/edit?usp=sharing), generated with kicad-footprint-generator")
+		(descr "LED SMD 0603 (1608 Metric), square (rectangular) end terminal, IPC_7351 nominal, (Body size source: http://www.tortai-tech.com/upload/download/2011102023233369053.pdf), generated with kicad-footprint-generator")
 		(tags "LED handsolder")
 		(property "Reference" "D1"
-			(at 0 -1.65 90)
+			(at 0 -1.43 -90)
 			(layer "F.SilkS")
-			(hide yes)
 			(effects
 				(font
@@
 		)
 		(property "Value" "PWR_Indicator"
-			(at 0 1.65 90)
+			(at 0 1.43 -90)
 			(layer "F.Fab")
 			(effects
@@
 			)
 		)
-		(property "Footprint" "LED_SMD:LED_0805_2012Metric_Pad1.15x1.40mm_HandSolder"
+		(property "Footprint" "LED_SMD:LED_0603_1608Metric_Pad1.05x0.95mm_HandSolder"
 			(at 0 0 -90)
 			(unlocked yes)
@@
 			)
 		)
-		(property "Part No" "C2297"
+		(property "Part No" "C125098"
 			(at 0 0 -90)
 			(unlocked yes)
@@
 			)
 		)
-		(property "Link" "https://www.lcsc.com/product-detail/LED-Indication-Discrete_Hubei-KENTO-Elec-KT-0805G_C2297.html"
+		(property "Link" "https://www.lcsc.com/product-detail/LED-Indication-Discrete_Lite-On-LTST-C191KGKT_C125098.html"
 			(at 0 0 -90)
 			(unlocked yes)
@@
 			)
 		)
-		(property "LCSC" "C2297"
+		(property "LCSC" "C125098"
 			(at 0 0 -90)
 			(unlocked yes)
@@
 		(attr smd)
 		(fp_line
-			(start -1.86 0.96)
-			(end 1 0.96)
+			(start -1.66 0.735)
+			(end 0.8 0.735)
 			(stroke
 				(width 0.12)
@@
 		)
 		(fp_line
-			(start -1.86 -0.96)
-			(end -1.86 0.96)
+			(start -1.66 -0.735)
+			(end -1.66 0.735)
 			(stroke
 				(width 0.12)
@@
 		)
 		(fp_line
-			(start 1 -0.96)
-			(end -1.86 -0.96)
+			(start 0.8 -0.735)
+			(end -1.66 -0.735)
 			(stroke
 				(width 0.12)
@@
 		)
 		(fp_line
-			(start -1.85 0.95)
-			(end -1.85 -0.95)
+			(start -1.65 0.73)
+			(end -1.65 -0.73)
 			(stroke
 				(width 0.05)
@@
 		)
 		(fp_line
-			(start 1.85 0.95)
-			(end -1.85 0.95)
+			(start 1.65 0.73)
+			(end -1.65 0.73)
 			(stroke
 				(width 0.05)
@@
 		)
 		(fp_line
-			(start -1.85 -0.95)
-			(end 1.85 -0.95)
+			(start -1.65 -0.73)
+			(end 1.65 -0.73)
 			(stroke
 				(width 0.05)
@@
 		)
 		(fp_line
-			(start 1.85 -0.95)
-			(end 1.85 0.95)
+			(start 1.65 -0.73)
+			(end 1.65 0.73)
 			(stroke
 				(width 0.05)
@@
 		)
 		(fp_line
-			(start -1 0.6)
-			(end 1 0.6)
+			(start -0.8 0.4)
+			(end 0.8 0.4)
 			(stroke
 				(width 0.1)
@@
 		)
 		(fp_line
-			(start 1 0.6)
-			(end 1 -0.6)
+			(start 0.8 0.4)
+			(end 0.8 -0.4)
 			(stroke
 				(width 0.1)
@@
 		)
 		(fp_line
-			(start -1 -0.3)
-			(end -1 0.6)
+			(start -0.8 -0.1)
+			(end -0.8 0.4)
 			(stroke
 				(width 0.1)
@@
 		)
 		(fp_line
-			(start -0.7 -0.6)
-			(end -1 -0.3)
+			(start -0.5 -0.4)
+			(end -0.8 -0.1)
 			(stroke
 				(width 0.1)
@@
 		)
 		(fp_line
-			(start 1 -0.6)
-			(end -0.7 -0.6)
+			(start 0.8 -0.4)
+			(end -0.5 -0.4)
 			(stroke
 				(width 0.1)
@@
 		)
 		(fp_text user "${REFERENCE}"
-			(at 0 0 90)
+			(at 0 0 -90)
 			(layer "F.Fab")
 			(effects
 				(font
-					(size 0.5 0.5)
-					(thickness 0.08)
+					(size 0.4 0.4)
+					(thickness 0.06)
 				)
 			)
 		)
 		(pad "1" smd roundrect
-			(at -1.025 0 270)
-			(size 1.15 1.4)
+			(at -0.875 0 270)
+			(size 1.05 0.95)
 			(layers "F.Cu" "F.Paste" "F.Mask")
-			(roundrect_rratio 0.217391)
+			(roundrect_rratio 0.25)
 			(net 14 "Net-(D1-K)")
 			(pinfunction "K")
@@
 		)
 		(pad "2" smd roundrect
-			(at 1.025 0 270)
-			(size 1.15 1.4)
+			(at 0.875 0 270)
+			(size 1.05 0.95)
 			(layers "F.Cu" "F.Paste" "F.Mask")
-			(roundrect_rratio 0.217391)
+			(roundrect_rratio 0.25)
 			(net 6 "+5V")
 			(pinfunction "A")
 			(pintype "passive")
 		)
-		(model "${KICAD8_3DMODEL_DIR}/LED_SMD.3dshapes/LED_0805_2012Metric.wrl"
+		(model "${KICAD8_3DMODEL_DIR}/LED_SMD.3dshapes/LED_0603_1608Metric.wrl"
 			(offset
 				(xyz 0 0 0)
@@
 		(tags "Power Jack")
 		(property "Reference" "J3"
-			(at -8.45 5.75 0)
+			(at -3 -3 0)
 			(layer "F.SilkS")
 			(effects
@@
 			)
 		)
-		(model "${KICAD8_3DMODEL_DIR}/Inductor_SMD.3dshapes/L_Coilcraft_LPS5030.wrl"
+		(model "/Users/peterhurd/Documents/KiCad/easyeda2kicad/easyeda2kicad.3dshapes/IND-SMD_L4.8-W4.8.step"
 			(offset
 				(xyz 0 0 0)
@@
 			(layer "F.SilkS")
 		)
+		(fp_poly
+			(pts
+				(xy -2.5 -2.575) (xy -2.74 -2.905) (xy -2.26 -2.905) (xy -2.5 -2.575)
+			)
+			(stroke
+				(width 0.12)
+				(type solid)
+			)
+			(fill solid)
+			(layer "F.SilkS")
+		)
 		(fp_line
 			(start 3.5 -2.55)
@@
 			(solder_paste_margin_ratio -0.2)
 		)
-		(model "${KICAD8_3DMODEL_DIR}/Package_SO.3dshapes/Diodes_SO-8EP.wrl"
+		(model "/Users/peterhurd/Documents/KiCad/easyeda2kicad/easyeda2kicad.3dshapes/SOP-8_L4.9-W3.9-H1.7-LS6.0-P1.30.step"
 			(offset
 				(xyz 0 0 0)
@@
 	(footprint "0_add_sub_module_tester:hurd_mark"
 		(layer "B.Cu")
-		(at 182 68.25 180)
+		(at 156.5 97.75 180)
 		(property "Reference" "REF**"
 			(at 0 -2.5 0)
@@
 	)
 	(gr_text "SDMAY25-29"
-		(at 207 71 0)
+		(at 197 101.5 0)
 		(layer "B.SilkS")
 		(effects
@@
 	)
 	(gr_text "Rev. A"
-		(at 204.000525 117.75 0)
+		(at 159.5 102.75 0)
 		(layer "B.SilkS")
 		(effects
@@
 	)
 	(gr_text "JLCJLCJLCJLC"
-		(at 207.499475 107.25 0)
+		(at 197.75 105.25 0)
 		(layer "B.SilkS")
 		(effects
@@
 		)
 	)
-	(gr_text "CARRY"
-		(at 154.5 74 0)
+	(gr_text "CARRY IN"
+		(at 157 74 0)
 		(layer "F.SilkS")
 		(effects
@@
 				(bold yes)
 			)
-			(justify left bottom)
+			(justify bottom)
 		)
 	)
@@
 	)
 	(gr_text "Rev. A"
-		(at 198.500525 117.75 0)
+		(at 154 102.75 0)
 		(layer "F.SilkS")
 		(effects
@@
 		)
 	)
-	(gr_text "KA"
-		(at 144 74 0)
+	(gr_text "Y/KA"
+		(at 145 74 0)
 		(layer "F.SilkS")
 		(effects
@@
 				(bold yes)
 			)
-			(justify left bottom)
+			(justify bottom)
+		)
+	)
+	(gr_text "+12VDC"
+		(at 135.5 105 0)
+		(layer "F.SilkS")
+		(effects
+			(font
+				(size 1 1)
+				(thickness 0.2)
+				(bold yes)
+			)
+			(justify bottom)
 		)
 	)
@@
 		)
 	)
-	(gr_text "CA"
-		(at 132 74 0)
+	(gr_text "X/CA"
+		(at 133 74 0)
 		(layer "F.SilkS")
 		(effects
@@
 				(bold yes)
 			)
-			(justify left bottom)
+			(justify bottom)
 		)
 	)
@@
 	)
 	(gr_text "PWR"
-		(at 132 93 90)
+		(at 128 89.5 0)
 		(layer "F.SilkS")
 		(effects
@@
 	)
 	(gr_text "Designed by:\nPeter Hurd"
-		(at 186.500525 102.25 0)
+		(at 152.5 98.5 0)
 		(layer "F.SilkS")
 		(effects
